File: ILJJ_Mk-XI.sch (KiCad schematic (older format))
At the start: 34 parts, among them J0 Conn_02x12_Odd_Even, J1 Conn_02x12_Odd_Even, J2 Conn_02x12_Odd_Even, J3 Conn_02x12_Odd_Even, J4 Conn_Input, J5 Conn_Output, SW0 SW_Coded_SH-7070, SW1 SW_Coded_SH-7070, SW2 SW_Coded_SH-7070, SW3 SW_Coded_SH-7070

Commit message: [add] Power indicator
Parts:
- added D?: LED, symbol Device:LED
- added R?: R, symbol Device:R
Changed lines of the file:
@@
 L power:GND #PWR?
 U 1 1 5C478506
-P 1050 1500
-F 0 "#PWR?" H 1050 1250 50  0001 C CNN
-F 1 "GND" H 1055 1327 50  0000 C CNN
-F 2 "" H 1050 1500 50  0001 C CNN
-F 3 "" H 1050 1500 50  0001 C CNN
-	1    1050 1500
+P 1050 1950
+F 0 "#PWR?" H 1050 1700 50  0001 C CNN
+F 1 "GND" H 1055 1777 50  0000 C CNN
+F 2 "" H 1050 1950 50  0001 C CNN
+F 3 "" H 1050 1950 50  0001 C CNN
+	1    1050 1950
 	1    0    0    -1
 $EndComp
@@
 L power:VCC #PWR?
 U 1 1 5C478569
-P 1050 1300
-F 0 "#PWR?" H 1050 1150 50  0001 C CNN
-F 1 "VCC" H 1067 1473 50  0000 C CNN
-F 2 "" H 1050 1300 50  0001 C CNN
-F 3 "" H 1050 1300 50  0001 C CNN
-	1    1050 1300
+P 1050 1350
+F 0 "#PWR?" H 1050 1200 50  0001 C CNN
+F 1 "VCC" H 1067 1523 50  0000 C CNN
+F 2 "" H 1050 1350 50  0001 C CNN
+F 3 "" H 1050 1350 50  0001 C CNN
+	1    1050 1350
 	1    0    0    -1
 $EndComp
@@
 L power:PWR_FLAG #FLG?
 U 1 1 5C4785DA
-P 1050 1300
-F 0 "#FLG?" H 1050 1375 50  0001 C CNN
-F 1 "PWR_FLAG" V 1050 1428 50  0000 L CNN
-F 2 "" H 1050 1300 50  0001 C CNN
-F 3 "~" H 1050 1300 50  0001 C CNN
-	1    1050 1300
-	0    1    1    0
+P 1050 1350
+F 0 "#FLG?" H 1050 1425 50  0001 C CNN
+F 1 "PWR_FLAG" V 1050 1478 50  0000 L CNN
+F 2 "" H 1050 1350 50  0001 C CNN
+F 3 "~" H 1050 1350 50  0001 C CNN
+	1    1050 1350
+	0    -1   -1   0
 $EndComp
 $Comp
 L power:PWR_FLAG #FLG?
 U 1 1 5C47860A
-P 1050 1500
-F 0 "#FLG?" H 1050 1575 50  0001 C CNN
-F 1 "PWR_FLAG" V 1050 1628 50  0000 L CNN
-F 2 "" H 1050 1500 50  0001 C CNN
-F 3 "~" H 1050 1500 50  0001 C CNN
-	1    1050 1500
-	0    1    1    0
+P 1050 1950
+F 0 "#FLG?" H 1050 2025 50  0001 C CNN
+F 1 "PWR_FLAG" V 1050 2078 50  0000 L CNN
+F 2 "" H 1050 1950 50  0001 C CNN
+F 3 "~" H 1050 1950 50  0001 C CNN
+	1    1050 1950
+	0    -1   -1   0
 $EndComp
 $Comp
@@
 Text Label 8300 4000 0    50   ~ 0
 S0
+$Comp
+L Device:R R?
+U 1 1 5C4FD83C
+P 1050 1500
+F 0 "R?" H 1120 1546 50  0000 L CNN
+F 1 "R" H 1120 1455 50  0000 L CNN
+F 2 "" V 980 1500 50  0001 C CNN
+F 3 "~" H 1050 1500 50  0001 C CNN
+	1    1050 1500
+	1    0    0    -1
+$EndComp
+Connection ~ 1050 1350
+$Comp
+L Device:LED D?
+U 1 1 5C4FD8E9
+P 1050 1800
+F 0 "D?" V 1088 1683 50  0000 R CNN
+F 1 "LED" V 997 1683 50  0000 R CNN
+F 2 "" H 1050 1800 50  0001 C CNN
+F 3 "~" H 1050 1800 50  0001 C CNN
+	1    1050 1800
+	0    -1   -1   0
+$EndComp
+Connection ~ 1050 1950
 $EndSCHEMATC

Commit message: [add] anotation
Parts:
- gave numbers to parts that had none: 26

Commit message: [add] some footprints
Parts:
- D0: footprint (none) -> LEDs:LED_D5.0mm
- D1, D2, D3, D4: footprint (none) -> LEDs:LED_Rectangular_W5.0mm_H2.0mm
- J4: footprint (none) -> Pin_Headers:Pin_Header_Angled_2x05_Pitch2.54mm
- J5: footprint (none) -> Socket_Strips:Socket_Strip_Angled_2x06_Pitch2.54mm
- SW0, SW1, SW2, SW3: footprint (none) -> Buttons_Switches_ThroughHole:Nidec_Copal_SH-7010C
Changed lines of the file:
@@
 F 0 "J4" H 8450 2767 50  0000 C CNN
 F 1 "Conn_Input" H 8450 2676 50  0000 C CNN
-F 2 "" H 8400 2350 50  0001 C CNN
+F 2 "Pin_Headers:Pin_Header_Angled_2x05_Pitch2.54mm" H 8400 2350 50  0001 C CNN
 F 3 "~" H 8400 2350 50  0001 C CNN
 	1    8400 2350
@@
 F 0 "J5" H 2650 2767 50  0000 C CNN
 F 1 "Conn_Output" H 2650 2676 50  0000 C CNN
-F 2 "" H 2600 2350 50  0001 C CNN
+F 2 "Socket_Strips:Socket_Strip_Angled_2x06_Pitch2.54mm" H 2600 2350 50  0001 C CNN
 F 3 "~" H 2600 2350 50  0001 C CNN
 	1    2600 2350
@@
 F 0 "SW3" H 3455 5967 50  0000 C CNN
 F 1 "SW_Coded_SH-7070" H 3455 5876 50  0000 C CNN
-F 2 "" H 3100 5050 50  0001 L CNN
+F 2 "Buttons_Switches_ThroughHole:Nidec_Copal_SH-7010C" H 3100 5050 50  0001 L CNN
 F 3 "https://www.nidec-copal-electronics.com/e/catalog/switch/sh-7000.pdf" H 3400 5500 50  0001 C CNN
 	1    3400 5500
@@
 F 0 "SW2" H 4555 5967 50  0000 C CNN
 F 1 "SW_Coded_SH-7070" H 4555 5876 50  0000 C CNN
-F 2 "" H 4200 5050 50  0001 L CNN
+F 2 "Buttons_Switches_ThroughHole:Nidec_Copal_SH-7010C" H 4200 5050 50  0001 L CNN
 F 3 "https://www.nidec-copal-electronics.com/e/catalog/switch/sh-7000.pdf" H 4500 5500 50  0001 C CNN
 	1    4500 5500
@@
 F 0 "SW1" H 3455 4967 50  0000 C CNN
 F 1 "SW_Coded_SH-7070" H 3455 4876 50  0000 C CNN
-F 2 "" H 3100 4050 50  0001 L CNN
+F 2 "Buttons_Switches_ThroughHole:Nidec_Copal_SH-7010C" H 3100 4050 50  0001 L CNN
 F 3 "https://www.nidec-copal-electronics.com/e/catalog/switch/sh-7000.pdf" H 3400 4500 50  0001 C CNN
 	1    3400 4500
@@
 F 0 "SW0" H 4555 4967 50  0000 C CNN
 F 1 "SW_Coded_SH-7070" H 4555 4876 50  0000 C CNN
-F 2 "" H 4200 4050 50  0001 L CNN
+F 2 "Buttons_Switches_ThroughHole:Nidec_Copal_SH-7010C" H 4200 4050 50  0001 L CNN
 F 3 "https://www.nidec-copal-electronics.com/e/catalog/switch/sh-7000.pdf" H 4500 4500 50  0001 C CNN
 	1    4500 4500
@@
 F 0 "D4" V 8245 4528 50  0000 L CNN
 F 1 "LED" V 8336 4528 50  0000 L CNN
-F 2 "" H 8300 4450 50  0001 C CNN
+F 2 "LEDs:LED_Rectangular_W5.0mm_H2.0mm" H 8300 4450 50  0001 C CNN
 F 3 "~" H 8300 4450 50  0001 C CNN
 	1    8300 4450
@@
 F 0 "D3" V 7895 4528 50  0000 L CNN
 F 1 "LED" V 7986 4528 50  0000 L CNN
-F 2 "" H 7950 4450 50  0001 C CNN
+F 2 "LEDs:LED_Rectangular_W5.0mm_H2.0mm" H 7950 4450 50  0001 C CNN
 F 3 "~" H 7950 4450 50  0001 C CNN
 	1    7950 4450
@@
 F 0 "D2" V 7545 4528 50  0000 L CNN
 F 1 "LED" V 7636 4528 50  0000 L CNN
-F 2 "" H 7600 4450 50  0001 C CNN
+F 2 "LEDs:LED_Rectangular_W5.0mm_H2.0mm" H 7600 4450 50  0001 C CNN
 F 3 "~" H 7600 4450 50  0001 C CNN
 	1    7600 4450
@@
 F 0 "D1" V 7195 4528 50  0000 L CNN
 F 1 "LED" V 7286 4528 50  0000 L CNN
-F 2 "" H 7250 4450 50  0001 C CNN
+F 2 "LEDs:LED_Rectangular_W5.0mm_H2.0mm" H 7250 4450 50  0001 C CNN
 F 3 "~" H 7250 4450 50  0001 C CNN
 	1    7250 4450
@@
 F 0 "D0" V 1688 2383 50  0000 R CNN
 F 1 "LED" V 1597 2383 50  0000 R CNN
-F 2 "" H 1650 2500 50  0001 C CNN
+F 2 "LEDs:LED_D5.0mm" H 1650 2500 50  0001 C CNN
 F 3 "~" H 1650 2500 50  0001 C CNN
 	1    1650 2500

Commit message: [change] interface connector
Parts:
- removed J4: Conn_Input, Pin_Headers:Pin_Header_Angled_2x05_Pitch2.54mm, symbol Connector_Generic:Conn_02x06_Row_Letter_Last
- removed J5: Conn_Output, Socket_Strips:Socket_Strip_Angled_2x06_Pitch2.54mm, symbol Connector_Generic:Conn_02x06_Row_Letter_Last
- added J4, J5: Conn_02x12_Row_Letter_Last, symbol Connector_Generic:Conn_02x12_Row_Letter_Last
Connections:
- wire segments 110 -> 118
Changed lines of the file:
@@
 EESchema Schematic File Version 4
+LIBS:ILJJ_Mk-XI-cache
 EELAYER 26 0
 EELAYER END
@@
 Wire Wire Line
 	7300 2500 7300 2550
-$Comp
-L Connector_Generic:Conn_02x06_Row_Letter_Last J4
-U 1 1 5C3E1736
-P 8400 2350
-F 0 "J4" H 8450 2767 50  0000 C CNN
-F 1 "Conn_Input" H 8450 2676 50  0000 C CNN
-F 2 "Pin_Headers:Pin_Header_Angled_2x05_Pitch2.54mm" H 8400 2350 50  0001 C CNN
-F 3 "~" H 8400 2350 50  0001 C CNN
-	1    8400 2350
-	1    0    0    -1
-$EndComp
-Wire Wire Line
-	8700 2150 8200 2150
 Connection ~ 7300 2150
-Connection ~ 8200 2150
-Wire Wire Line
-	8200 2150 7300 2150
-Wire Wire Line
-	8700 2250 8200 2250
 Connection ~ 7300 2250
-Connection ~ 8200 2250
-Wire Wire Line
-	8200 2250 7300 2250
-Wire Wire Line
-	8700 2350 8200 2350
 Connection ~ 7300 2350
-Connection ~ 8200 2350
-Wire Wire Line
-	8200 2350 7300 2350
-Wire Wire Line
-	8700 2450 8200 2450
 Connection ~ 7300 2450
-Connection ~ 8200 2450
-Wire Wire Line
-	8200 2450 7300 2450
 Wire Wire Line
 	6800 2550 6800 2600
@@
 Wire Wire Line
 	7350 2600 7350 2550
-Wire Wire Line
-	7350 2550 8200 2550
-Connection ~ 8200 2550
-Wire Wire Line
-	8200 2550 8700 2550
-Wire Wire Line
-	8700 2650 8200 2650
-Connection ~ 7300 2650
-Connection ~ 8200 2650
-Wire Wire Line
-	8200 2650 7300 2650
-$Comp
-L Connector_Generic:Conn_02x06_Row_Letter_Last J5
-U 1 1 5C3E925F
-P 2600 2350
-F 0 "J5" H 2650 2767 50  0000 C CNN
-F 1 "Conn_Output" H 2650 2676 50  0000 C CNN
-F 2 "Socket_Strips:Socket_Strip_Angled_2x06_Pitch2.54mm" H 2600 2350 50  0001 C CNN
-F 3 "~" H 2600 2350 50  0001 C CNN
-	1    2600 2350
-	1    0    0    -1
-$EndComp
-Wire Wire Line
-	2400 2150 2900 2150
 Connection ~ 3800 2150
-Connection ~ 2900 2150
-Wire Wire Line
-	2900 2150 3800 2150
-Wire Wire Line
-	2400 2250 2900 2250
 Connection ~ 3800 2250
-Connection ~ 2900 2250
-Wire Wire Line
-	2900 2250 3800 2250
-Wire Wire Line
-	2400 2350 2900 2350
 Connection ~ 3800 2350
-Connection ~ 2900 2350
-Wire Wire Line
-	2900 2350 3800 2350
-Wire Wire Line
-	2400 2450 2900 2450
 Connection ~ 3800 2450
-Connection ~ 2900 2450
-Wire Wire Line
-	2900 2450 3800 2450
 Wire Wire Line
 	4300 2550 4300 2600
@@
 Wire Wire Line
 	3750 2600 3750 2550
-Wire Wire Line
-	3750 2550 2900 2550
-Wire Wire Line
-	2400 2550 2900 2550
-Connection ~ 2900 2550
-Wire Wire Line
-	2400 2650 2900 2650
-Connection ~ 3800 2650
-Connection ~ 2900 2650
-Wire Wire Line
-	2900 2650 3800 2650
 Text Label 6800 3250 2    50   ~ 0
 A0
@@
 L power:VCC #PWR09
 U 1 1 5C458F94
-P 8850 1950
-F 0 "#PWR09" H 8850 1800 50  0001 C CNN
-F 1 "VCC" H 8867 2123 50  0000 C CNN
-F 2 "" H 8850 1950 50  0001 C CNN
-F 3 "" H 8850 1950 50  0001 C CNN
-	1    8850 1950
+P 8200 1950
+F 0 "#PWR09" H 8200 1800 50  0001 C CNN
+F 1 "VCC" H 8217 2123 50  0000 C CNN
+F 2 "" H 8200 1950 50  0001 C CNN
+F 3 "" H 8200 1950 50  0001 C CNN
+	1    8200 1950
 	1    0    0    -1
 $EndComp
@@
 L power:GND #PWR010
 U 1 1 5C459007
-P 8850 2850
-F 0 "#PWR010" H 8850 2600 50  0001 C CNN
-F 1 "GND" H 8855 2677 50  0000 C CNN
-F 2 "" H 8850 2850 50  0001 C CNN
-F 3 "" H 8850 2850 50  0001 C CNN
-	1    8850 2850
-	1    0    0    -1
-$EndComp
-Wire Wire Line
-	8700 2150 8850 2150
-Wire Wire Line
-	8850 2150 8850 1950
-Connection ~ 8700 2150
-Wire Wire Line
-	8700 2650 8850 2650
-Wire Wire Line
-	8850 2650 8850 2850
-Connection ~ 8700 2650
+P 8200 3450
+F 0 "#PWR010" H 8200 3200 50  0001 C CNN
+F 1 "GND" H 8205 3277 50  0000 C CNN
+F 2 "" H 8200 3450 50  0001 C CNN
+F 3 "" H 8200 3450 50  0001 C CNN
+	1    8200 3450
+	1    0    0    -1
+$EndComp
+Wire Wire Line
+	8200 2150 8200 1950
 Text Label 6300 3250 0    50   ~ 0
 B2
@@
 $EndComp
 Connection ~ 1650 2650
+Wire Wire Line
+	7300 2150 8200 2150
+$Comp
+L Connector_Generic:Conn_02x12_Row_Letter_Last J4
+U 1 1 5C481A6C
+P 8750 2650
+F 0 "J4" H 8800 3367 50  0000 C CNN
+F 1 "Conn_02x12_Row_Letter_Last" H 8800 3276 50  0000 C CNN
+F 2 "" H 8750 2650 50  0001 C CNN
+F 3 "~" H 8750 2650 50  0001 C CNN
+	1    8750 2650
+	1    0    0    -1
+$EndComp
+Wire Wire Line
+	7300 2650 8200 2650
+Wire Wire Line
+	8200 2650 8200 3250
+Connection ~ 7300 2650
+Connection ~ 8550 3250
+Wire Wire Line
+	8550 3250 9050 3250
+Wire Wire Line
+	7350 2550 8300 2550
+Wire Wire Line
+	8300 2550 8300 3050
+Wire Wire Line
+	8300 3050 8550 3050
+Connection ~ 8550 3050
+Wire Wire Line
+	8550 3050 9050 3050
+Wire Wire Line
+	7300 2450 8550 2450
+Connection ~ 8550 2450
+Wire Wire Line
+	8550 2450 9050 2450
+Wire Wire Line
+	7300 2350 8550 2350
+Connection ~ 8550 2350
+Wire Wire Line
+	8550 2350 9050 2350
+Wire Wire Line
+	7300 2250 8550 2250
+Connection ~ 8550 2250
+Wire Wire Line
+	8550 2250 9050 2250
+Wire Wire Line
+	9050 2150 8550 2150
+Connection ~ 8200 2150
+Connection ~ 8550 2150
+Wire Wire Line
+	8550 2150 8200 2150
+Wire Wire Line
+	8200 3250 8200 3450
+Connection ~ 8200 3250
+Wire Wire Line
+	8200 3250 8550 3250
+Connection ~ 8200 3450
+Wire Wire Line
+	8200 3450 8200 3550
+$Comp
+L Connector_Generic:Conn_02x12_Row_Letter_Last J5
+U 1 1 5C4ACF80
+P 2600 2650
+F 0 "J5" H 2650 3367 50  0000 C CNN
+F 1 "Conn_02x12_Row_Letter_Last" H 2650 3276 50  0000 C CNN
+F 2 "" H 2600 2650 50  0001 C CNN
+F 3 "~" H 2600 2650 50  0001 C CNN
+	1    2600 2650
+	1    0    0    -1
+$EndComp
+Wire Wire Line
+	2900 2150 3800 2150
+Wire Wire Line
+	2900 2350 3800 2350
+Wire Wire Line
+	2900 2450 3800 2450
+Wire Wire Line
+	2400 2150 2900 2150
+Connection ~ 2900 2150
+Wire Wire Line
+	2400 2250 2900 2250
+Connection ~ 2900 2250
+Wire Wire Line
+	2900 2250 3800 2250
+Wire Wire Line
+	2400 2350 2900 2350
+Connection ~ 2900 2350
+Wire Wire Line
+	2400 2450 2900 2450
+Connection ~ 2900 2450
+Wire Wire Line
+	3750 2550 3500 2550
+Wire Wire Line
+	3800 2650 3600 2650
+Wire Wire Line
+	3600 2650 3600 3250
+Wire Wire Line
+	3600 3250 2900 3250
+Connection ~ 3800 2650
+Connection ~ 2900 3250
+Wire Wire Line
+	2900 3250 2400 3250
+Wire Wire Line
+	3500 2550 3500 3050
+Wire Wire Line
+	3500 3050 2900 3050
+Connection ~ 2900 3050
+Wire Wire Line
+	2900 3050 2400 3050
 $EndSCHEMATC

Commit message: [add] buffer for function pin
Parts:
- added U1, U2, U3: 7400, symbol 74xx:7400
Connections:
- net labels added: F0, F0_1, F0_2, F1, F1_1, F1_2, F2, F2_1, F2_2
- wire segments 118 -> 150
Other:
- moved on the sheet: SW0, SW1, SW2, SW3

Commit message: [add] footprint for card edge connector socket
Parts:
- J0, J1, J2, J3: footprint (none) -> fplib:5530843-1_socket
- J4: footprint (none) -> Pin_Headers:Pin_Header_Angled_2x12_Pitch2.54mm
- J5: footprint (none) -> Socket_Strips:Socket_Strip_Angled_2x12_Pitch2.54mm
- R0, R1, R10, R11, R12, R13, R14, R15, R16, R17, R18, R19, R2, R20, R3, R4, R5, R6, R7, R8, R9: footprint (none) -> Resistors_ThroughHole:R_Axial_DIN0204_L3.6mm_D1.6mm_P2.54mm_Vertical
- U1, U2, U3: footprint (none) -> Housings_DIP:DIP-14_W7.62mm_LongPads

Commit message: [add] input indicator
Parts:
- added D10, D11, D12, D13, D14, D15, D16, D17, D18, D19, D20, D5, D6, D7, D8, D9: LED, LEDs:LED_Rectangular_W5.0mm_H2.0mm, symbol Device:LED
- added R21, R22, R23, R24, R25, R26, R27, R28, R29, R30, R31, R32, R33, R34, R35, R36: R, Resistors_ThroughHole:R_Axial_DIN0204_L3.6mm_D1.6mm_P2.54mm_Vertical, symbol Device:R
Other:
- moved on the sheet: SW0, SW1, SW2, SW3, U1A, U1B, U1C, U1D, U2A, U2B, U2C, U2D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

Commit message: [fix] 出力LEDが4bitしかなかった
なんで気付かなかったんだろう...
Parts:
- added D21, D22, D23, D24: LED, LEDs:LED_Rectangular_W5.0mm_H2.0mm, symbol Device:LED
- added R37, R38, R39, R40: R, Resistors_ThroughHole:R_Axial_DIN0204_L3.6mm_D1.6mm_P2.54mm_Vertical, symbol Device:R
Connections:
- wire segments 150 -> 161
- no-connect marks 24 -> 48
