File: ILJJ_Mk-XI.sch (KiCad schematic (older format))
At the start: 79 parts, among them J0 Conn_02x12_Odd_Even, J1 Conn_02x12_Odd_Even, J2 Conn_02x12_Odd_Even, J3 Conn_02x12_Odd_Even, J4 Conn_02x12_Row_Letter_Last, J5 Conn_02x12_Row_Letter_Last, SW0 SW_Coded_SH-7070, SW1 SW_Coded_SH-7070, SW2 SW_Coded_SH-7070, SW3 SW_Coded_SH-7070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

Commit message: [fix] コネクタのコンポーネントを変更
Parts:
- removed J4: Conn_02x12_Row_Letter_Last, Pin_Headers:Pin_Header_Angled_2x12_Pitch2.54mm, symbol Connector_Generic:Conn_02x12_Row_Letter_Last
- removed J5: Conn_02x12_Row_Letter_Last, Socket_Strips:Socket_Strip_Angled_2x12_Pitch2.54mm, symbol Connector_Generic:Conn_02x12_Row_Letter_Last
- added J4: Conn_02x12_Odd_Even, Pin_Headers:Pin_Header_Straight_2x12_Pitch2.54mm, symbol Connector_Generic:Conn_02x12_Odd_Even
- added J5: Conn_02x12_Odd_Even, Socket_Strips:Socket_Strip_Straight_2x12_Pitch2.54mm, symbol Connector_Generic:Conn_02x12_Odd_Even
Changed lines of the file:
@@
 Wire Wire Line
 	7300 2150 8200 2150
-$Comp
-L Connector_Generic:Conn_02x12_Row_Letter_Last J4
-U 1 1 5C481A6C
-P 8750 2650
-F 0 "J4" H 8800 3367 50  0000 C CNN
-F 1 "Conn_02x12_Row_Letter_Last" H 8800 3276 50  0000 C CNN
-F 2 "Pin_Headers:Pin_Header_Angled_2x12_Pitch2.54mm" H 8750 2650 50  0001 C CNN
-F 3 "~" H 8750 2650 50  0001 C CNN
-	1    8750 2650
-	1    0    0    -1
-$EndComp
 Wire Wire Line
 	7300 2650 8200 2650
@@
 	8200 2650 8200 3250
 Connection ~ 7300 2650
-Connection ~ 8550 3250
-Wire Wire Line
-	8550 3250 9050 3250
 Wire Wire Line
 	7350 2550 8300 2550
 Wire Wire Line
 	8300 2550 8300 3050
-Wire Wire Line
-	8300 3050 8550 3050
-Connection ~ 8550 3050
-Wire Wire Line
-	8550 3050 9050 3050
-Wire Wire Line
-	8550 2450 9050 2450
-Wire Wire Line
-	8550 2350 9050 2350
-Wire Wire Line
-	8550 2250 9050 2250
-Wire Wire Line
-	9050 2150 8550 2150
 Connection ~ 8200 2150
-Connection ~ 8550 2150
-Wire Wire Line
-	8550 2150 8200 2150
 Wire Wire Line
 	8200 3250 8200 3450
 Connection ~ 8200 3250
 Wire Wire Line
-	8200 3250 8550 3250
-$Comp
-L Connector_Generic:Conn_02x12_Row_Letter_Last J5
-U 1 1 5C4ACF80
-P 2600 2650
-F 0 "J5" H 2650 3367 50  0000 C CNN
-F 1 "Conn_02x12_Row_Letter_Last" H 2650 3276 50  0000 C CNN
-F 2 "Socket_Strips:Socket_Strip_Angled_2x12_Pitch2.54mm" H 2600 2650 50  0001 C CNN
-F 3 "~" H 2600 2650 50  0001 C CNN
-	1    2600 2650
-	1    0    0    -1
-$EndComp
-Wire Wire Line
-	2900 2150 3800 2150
-Wire Wire Line
-	2400 2150 2900 2150
-Connection ~ 2900 2150
-Wire Wire Line
-	2400 2250 2900 2250
-Wire Wire Line
-	2400 2350 2900 2350
-Wire Wire Line
-	2400 2450 2900 2450
-Wire Wire Line
 	3750 2550 3500 2550
 Wire Wire Line
@@
 Wire Wire Line
 	3600 2650 3600 3250
-Wire Wire Line
-	3600 3250 2900 3250
 Connection ~ 3800 2650
-Connection ~ 2900 3250
-Wire Wire Line
-	2900 3250 2400 3250
 Wire Wire Line
 	3500 2550 3500 3050
-Wire Wire Line
-	3500 3050 2900 3050
-Connection ~ 2900 3050
-Wire Wire Line
-	2900 3050 2400 3050
 $Comp
 L 74xx:7400 U1
@@
 NoConn ~ 2400 2950
 NoConn ~ 2400 3150
-Wire Wire Line
-	2900 2250 3800 2250
-Connection ~ 2900 2250
 Connection ~ 3800 2250
-Wire Wire Line
-	2900 2350 3800 2350
-Connection ~ 2900 2350
 Connection ~ 3800 2350
-Wire Wire Line
-	2900 2450 3800 2450
-Connection ~ 2900 2450
 Connection ~ 3800 2450
 $Comp
@@
 Text Label 2950 6750 0    50   ~ 0
 B7
+Wire Wire Line
+	8300 3050 8550 3050
+Wire Wire Line
+	8200 3250 8550 3250
+Wire Wire Line
+	8200 2150 8550 2150
+$Comp
+L Connector_Generic:Conn_02x12_Odd_Even J4
+U 1 1 5C70FF81
+P 8750 2650
+F 0 "J4" H 8800 3367 50  0000 C CNN
+F 1 "Conn_02x12_Odd_Even" H 8800 3276 50  0000 C CNN
+F 2 "Pin_Headers:Pin_Header_Straight_2x12_Pitch2.54mm" H 8750 2650 50  0001 C CNN
+F 3 "~" H 8750 2650 50  0001 C CNN
+	1    8750 2650
+	1    0    0    -1
+$EndComp
+Wire Wire Line
+	8550 2150 9050 2150
+Connection ~ 8550 2150
+Wire Wire Line
+	8550 3050 9050 3050
+Connection ~ 8550 3050
+Wire Wire Line
+	8550 3250 9050 3250
+Connection ~ 8550 3250
+Wire Wire Line
+	8550 2250 9050 2250
+Wire Wire Line
+	8550 2350 9050 2350
+Wire Wire Line
+	8550 2450 9050 2450
+$Comp
+L Connector_Generic:Conn_02x12_Odd_Even J5
+U 1 1 5C734624
+P 2600 2650
+F 0 "J5" H 2650 3367 50  0000 C CNN
+F 1 "Conn_02x12_Odd_Even" H 2650 3276 50  0000 C CNN
+F 2 "Socket_Strips:Socket_Strip_Straight_2x12_Pitch2.54mm" H 2600 2650 50  0001 C CNN
+F 3 "~" H 2600 2650 50  0001 C CNN
+	1    2600 2650
+	1    0    0    -1
+$EndComp
+Wire Wire Line
+	2900 2150 3800 2150
+Wire Wire Line
+	2900 3050 3500 3050
+Wire Wire Line
+	2900 3250 3600 3250
+Wire Wire Line
+	2900 2250 3800 2250
+Wire Wire Line
+	2900 2350 3800 2350
+Wire Wire Line
+	2900 2450 3800 2450
+Wire Wire Line
+	2400 2150 2900 2150
+Connection ~ 2900 2150
+Wire Wire Line
+	2400 2250 2900 2250
+Connection ~ 2900 2250
+Wire Wire Line
+	2400 2350 2900 2350
+Connection ~ 2900 2350
+Wire Wire Line
+	2400 2450 2900 2450
+Connection ~ 2900 2450
+Wire Wire Line
+	2400 3050 2900 3050
+Connection ~ 2900 3050
+Wire Wire Line
+	2400 3250 2900 3250
+Connection ~ 2900 3250
 $EndSCHEMATC

Commit message: [add] pcb
Parts:
- added unit 5 of U1
- added unit 5 of U2
- added unit 5 of U3
Connections:
- wire segments 161 -> 165
Changed lines of the file:
@@
 $Comp
 L 74xx:7400 U1
-U 2 1 5C578F10
+U 4 1 5C578F10
 P 6000 4050
 F 0 "U1" H 6000 4375 50  0000 C CNN
@@
 F 2 "Housings_DIP:DIP-14_W7.62mm_LongPads" H 6000 4050 50  0001 C CNN
 F 3 "http://www.ti.com/lit/gpn/sn7400" H 6000 4050 50  0001 C CNN
-	2    6000 4050
+	4    6000 4050
 	1    0    0    -1
 $EndComp
@@
 $Comp
 L 74xx:7400 U2
-U 2 1 5C579033
+U 4 1 5C579033
 P 6000 4700
 F 0 "U2" H 6000 5025 50  0000 C CNN
@@
 F 2 "Housings_DIP:DIP-14_W7.62mm_LongPads" H 6000 4700 50  0001 C CNN
 F 3 "http://www.ti.com/lit/gpn/sn7400" H 6000 4700 50  0001 C CNN
-	2    6000 4700
+	4    6000 4700
 	1    0    0    -1
 $EndComp
@@
 $Comp
 L 74xx:7400 U3
-U 2 1 5C57B374
+U 4 1 5C57B374
 P 6000 5300
 F 0 "U3" H 6000 5625 50  0000 C CNN
@@
 F 2 "Housings_DIP:DIP-14_W7.62mm_LongPads" H 6000 5300 50  0001 C CNN
 F 3 "http://www.ti.com/lit/gpn/sn7400" H 6000 5300 50  0001 C CNN
-	2    6000 5300
+	4    6000 5300
 	1    0    0    -1
 $EndComp
 $Comp
 L 74xx:7400 U1
-U 3 1 5C57D6B2
+U 2 1 5C57D6B2
 P 6800 4050
 F 0 "U1" H 6800 4375 50  0000 C CNN
@@
 F 2 "Housings_DIP:DIP-14_W7.62mm_LongPads" H 6800 4050 50  0001 C CNN
 F 3 "http://www.ti.com/lit/gpn/sn7400" H 6800 4050 50  0001 C CNN
-	3    6800 4050
+	2    6800 4050
 	1    0    0    -1
 $EndComp
 $Comp
 L 74xx:7400 U1
-U 4 1 5C57D6B9
+U 3 1 5C57D6B9
 P 7400 4050
 F 0 "U1" H 7400 4375 50  0000 C CNN
@@
 F 2 "Housings_DIP:DIP-14_W7.62mm_LongPads" H 7400 4050 50  0001 C CNN
 F 3 "http://www.ti.com/lit/gpn/sn7400" H 7400 4050 50  0001 C CNN
-	4    7400 4050
+	3    7400 4050
 	1    0    0    -1
 $EndComp
 $Comp
 L 74xx:7400 U2
-U 3 1 5C58418B
+U 2 1 5C58418B
 P 6800 4700
 F 0 "U2" H 6800 5025 50  0000 C CNN
@@
 F 2 "Housings_DIP:DIP-14_W7.62mm_LongPads" H 6800 4700 50  0001 C CNN
 F 3 "http://www.ti.com/lit/gpn/sn7400" H 6800 4700 50  0001 C CNN
-	3    6800 4700
+	2    6800 4700
 	1    0    0    -1
 $EndComp
 $Comp
 L 74xx:7400 U2
-U 4 1 5C584192
+U 3 1 5C584192
 P 7400 4700
 F 0 "U2" H 7400 5025 50  0000 C CNN
@@
 F 2 "Housings_DIP:DIP-14_W7.62mm_LongPads" H 7400 4700 50  0001 C CNN
 F 3 "http://www.ti.com/lit/gpn/sn7400" H 7400 4700 50  0001 C CNN
-	4    7400 4700
+	3    7400 4700
 	1    0    0    -1
 $EndComp
 $Comp
 L 74xx:7400 U3
-U 3 1 5C5864CC
+U 2 1 5C5864CC
 P 6800 5300
 F 0 "U3" H 6800 5625 50  0000 C CNN
@@
 F 2 "Housings_DIP:DIP-14_W7.62mm_LongPads" H 6800 5300 50  0001 C CNN
 F 3 "http://www.ti.com/lit/gpn/sn7400" H 6800 5300 50  0001 C CNN
-	3    6800 5300
+	2    6800 5300
 	1    0    0    -1
 $EndComp
 $Comp
 L 74xx:7400 U3
-U 4 1 5C5864D3
+U 3 1 5C5864D3
 P 7400 5300
 F 0 "U3" H 7400 5625 50  0000 C CNN
@@
 F 2 "Housings_DIP:DIP-14_W7.62mm_LongPads" H 7400 5300 50  0001 C CNN
 F 3 "http://www.ti.com/lit/gpn/sn7400" H 7400 5300 50  0001 C CNN
-	4    7400 5300
+	3    7400 5300
 	1    0    0    -1
 $EndComp
@@
 	2400 3250 2900 3250
 Connection ~ 2900 3250
+$Comp
+L 74xx:7400 U1
+U 5 1 5C79836F
+P 8500 5500
+F 0 "U1" H 8730 5546 50  0000 L CNN
+F 1 "7400" H 8730 5455 50  0000 L CNN
+F 2 "" H 8500 5500 50  0001 C CNN
+F 3 "http://www.ti.com/lit/gpn/sn7400" H 8500 5500 50  0001 C CNN
+	5    8500 5500
+	1    0    0    -1
+$EndComp
+$Comp
+L 74xx:7400 U2
+U 5 1 5C798BB2
+P 9200 5500
+F 0 "U2" H 9430 5546 50  0000 L CNN
+F 1 "7400" H 9430 5455 50  0000 L CNN
+F 2 "" H 9200 5500 50  0001 C CNN
+F 3 "http://www.ti.com/lit/gpn/sn7400" H 9200 5500 50  0001 C CNN
+	5    9200 5500
+	1    0    0    -1
+$EndComp
+$Comp
+L 74xx:7400 U3
+U 5 1 5C798C82
+P 9900 5500
+F 0 "U3" H 10130 5546 50  0000 L CNN
+F 1 "7400" H 10130 5455 50  0000 L CNN
+F 2 "" H 9900 5500 50  0001 C CNN
+F 3 "http://www.ti.com/lit/gpn/sn7400" H 9900 5500 50  0001 C CNN
+	5    9900 5500
+	1    0    0    -1
+$EndComp
+Wire Wire Line
+	8500 5000 9200 5000
+Connection ~ 9200 5000
+Wire Wire Line
+	9200 5000 9900 5000
+Wire Wire Line
+	8500 6000 9200 6000
+Connection ~ 9200 6000
+Wire Wire Line
+	9200 6000 9900 6000
+$Comp
+L power:GND #PWR028
+U 1 1 5C7A6C0C
+P 9900 6000
+F 0 "#PWR028" H 9900 5750 50  0001 C CNN
+F 1 "GND" H 9905 5827 50  0000 C CNN
+F 2 "" H 9900 6000 50  0001 C CNN
+F 3 "" H 9900 6000 50  0001 C CNN
+	1    9900 6000
+	1    0    0    -1
+$EndComp
+Connection ~ 9900 6000
+$Comp
+L power:VCC #PWR027
+U 1 1 5C7A6E26
+P 8500 5000
+F 0 "#PWR027" H 8500 4850 50  0001 C CNN
+F 1 "VCC" H 8517 5173 50  0000 C CNN
+F 2 "" H 8500 5000 50  0001 C CNN
+F 3 "" H 8500 5000 50  0001 C CNN
+	1    8500 5000
+	1    0    0    -1
+$EndComp
+Connection ~ 8500 5000
 $EndSCHEMATC

Commit message: [change] バッファの配線を変更
まあ元の配線がどう考えてもおかしい
Connections:
- wire segments 165 -> 156
Changed lines of the file:
@@
 Wire Wire Line
 	7350 2600 7350 2550
-Connection ~ 3800 2150
 Wire Wire Line
 	4300 2550 4300 2600
@@
 F2
 Wire Wire Line
-	6500 3950 6500 4050
-Wire Wire Line
-	6300 4050 6400 4050
-Connection ~ 6500 4050
-Wire Wire Line
-	6500 4050 6500 4150
-Wire Wire Line
-	6500 4600 6500 4700
-Wire Wire Line
 	6300 4700 6400 4700
-Connection ~ 6500 4700
-Wire Wire Line
-	6500 4700 6500 4800
-Wire Wire Line
-	6500 5200 6500 5300
 Wire Wire Line
 	6300 5300 6400 5300
-Connection ~ 6500 5300
-Wire Wire Line
-	6500 5300 6500 5400
 Wire Wire Line
 	5100 3950 5100 4050
@@
 F0
 Wire Wire Line
-	6400 4050 6400 3950
-Connection ~ 6400 4050
-Wire Wire Line
-	6400 4050 6500 4050
-Wire Wire Line
 	6400 4700 6400 4600
-Connection ~ 6400 4700
-Wire Wire Line
-	6400 4700 6500 4700
 Wire Wire Line
 	6400 5300 6400 5200
-Connection ~ 6400 5300
-Wire Wire Line
-	6400 5300 6500 5300
 Text Label 6400 3950 1    50   ~ 0
 F2_1
@@
 NoConn ~ 2400 2950
 NoConn ~ 2400 3150
-Connection ~ 3800 2250
-Connection ~ 3800 2350
-Connection ~ 3800 2450
 $Comp
 L Device:LED D4
@@
 $EndComp
 Wire Wire Line
-	2900 2150 3800 2150
-Wire Wire Line
 	2900 3050 3500 3050
 Wire Wire Line
 	2900 3250 3600 3250
 Wire Wire Line
-	2900 2250 3800 2250
-Wire Wire Line
-	2900 2350 3800 2350
-Wire Wire Line
-	2900 2450 3800 2450
-Wire Wire Line
 	2400 2150 2900 2150
-Connection ~ 2900 2150
 Wire Wire Line
 	2400 2250 2900 2250
-Connection ~ 2900 2250
 Wire Wire Line
 	2400 2350 2900 2350
-Connection ~ 2900 2350
 Wire Wire Line
 	2400 2450 2900 2450
-Connection ~ 2900 2450
 Wire Wire Line
 	2400 3050 2900 3050
@@
 $EndComp
 Connection ~ 8500 5000
+Connection ~ 3800 2150
+Connection ~ 2900 2150
+Wire Wire Line
+	2900 2150 3800 2150
+Text Label 2900 2250 0    50   ~ 0
+F2
+Text Label 2900 2350 0    50   ~ 0
+F1
+Text Label 2900 2450 0    50   ~ 0
+F0
+Wire Wire Line
+	6500 3950 6500 4150
+Wire Wire Line
+	6300 4050 6400 4050
+Wire Wire Line
+	6400 4050 6400 3950
+Wire Wire Line
+	6500 4600 6500 4800
+Wire Wire Line
+	6500 5200 6500 5400
+Text Label 6500 3950 1    50   ~ 0
+F2
+Text Label 6500 4600 1    50   ~ 0
+F1
+Text Label 6500 5200 1    50   ~ 0
+F0
 $EndSCHEMATC
